Commit message: ee added

File: onelink_robot/urdf/onelink_robot_support_macro.xacro (robot description, xacro)
@@ -3,60 +3,150 @@
   <xacro:macro name="onelink_robot" params="prefix">
     <!-- links: main serial chain -->
-  <link name="${prefix}base_link">
-      <inertial>
-        <origin xyz="8.7018E-07 2.7995E-08 0.047164" rpy="0 0 0" />
-        <mass value="1.3101" />
-        <inertia ixx="0.0024623" ixy="3.2088E-09" ixz="2.422E-09"
-          iyy="0.0024625" iyz="-4.6557E-09"
-          izz="0.0027581" />
-      </inertial>
-      <visual>
-        <origin xyz="0 0 0" rpy="0 0 0" />
-        <geometry>
-          <mesh filename="package://onelink_robot/meshes/visual/base_link.STL" />
-        </geometry>
-        <material
-          name="">
-          <color rgba="0.79216 0.81961 0.93333 1" />
-        </material>
-      </visual>
-      <collision>
-        <origin xyz="0 0 0" rpy="0 0 0" />
-        <geometry>
-          <mesh filename="package://onelink_robot/meshes/collision/base_link.STL" />
-        </geometry>
-      </collision>
-    </link>
-    <link name="${prefix}link_1">
-      <inertial>
-        <origin xyz="-0.30846 -0.007069 -0.0093247" rpy="0 0 0" />
-        <mass value="4.5602" />
-        <inertia ixx="0.0089629" ixy="-0.001234" ixz="-0.0059844"
-          iyy="0.06278" iyz="-0.00013714"
-          izz="0.061068" />
-      </inertial>
-      <visual>
-        <origin xyz="0 0 0" rpy="0 0 0" />
-        <geometry>
-          <mesh filename="package://onelink_robot/meshes/visual/link_1.STL" />
-        </geometry>
-        <material name="">
-          <color rgba="1 0.93725 0.13725 1" />
-        </material>
-      </visual>
-      <collision>
-        <origin xyz="0 0 0" rpy="0 0 0" />
-        <geometry>
-          <mesh filename="package://onelink_robot/meshes/collision/link_1.STL" />
-        </geometry>
-      </collision>
-    </link>
-    <joint name="${prefix}joint_1" type="continuous">
-      <origin xyz="0.45811 0.010499 0.195" rpy="0 0 0" />
-      <parent link="${prefix}base_link" />
-      <child link="${prefix}link_1" />
-      <axis xyz="0 0 1" />
-      <dynamics damping="0.0" friction="0.0"/>
-    </joint>
+  <link
+    name="${prefix}base_link">
+    <inertial>
+      <origin
+        xyz="8.7018E-07 2.7995E-08 0.047164"
+        rpy="0 0 0" />
+      <mass
+        value="1.3101" />
+      <inertia
+        ixx="0.0024623"
+        ixy="3.2088E-09"
+        ixz="2.422E-09"
+        iyy="0.0024625"
+        iyz="-4.6557E-09"
+        izz="0.0027581" />
+    </inertial>
+    <visual>
+      <origin
+        xyz="0 0 0"
+        rpy="0 0 0" />
+      <geometry>
+        <mesh
+          filename="package://onelink_robot/meshes/base_link.STL" />
+      </geometry>
+      <material
+        name="">
+        <color
+          rgba="0.79216 0.81961 0.93333 1" />
+      </material>
+    </visual>
+    <collision>
+      <origin
+        xyz="0 0 0"
+        rpy="0 0 0" />
+      <geometry>
+        <mesh
+          filename="package://onelink_robot/meshes/base_link.STL" />
+      </geometry>
+    </collision>
+  </link>
+  <link
+    name="${prefix}link_1">
+    <inertial>
+      <origin
+        xyz="0.13171 0.040866 0.085302"
+        rpy="0 0 0" />
+      <mass
+        value="4.3846" />
+      <inertia
+        ixx="0.013596"
+        ixy="-0.015233"
+        ixz="-0.0057172"
+        iyy="0.057965"
+        iyz="-0.0017739"
+        izz="0.060952" />
+    </inertial>
+    <visual>
+      <origin
+        xyz="0 0 0"
+        rpy="0 0 0" />
+      <geometry>
+        <mesh
+          filename="package://onelink_robot/meshes/link_1.STL" />
+      </geometry>
+      <material
+        name="">
+        <color
+          rgba="1 0.93725 0.13725 1" />
+      </material>
+    </visual>
+    <collision>
+      <origin
+        xyz="0 0 0"
+        rpy="0 0 0" />
+      <geometry>
+        <mesh
+          filename="package://onelink_robot/meshes/link_1.STL" />
+      </geometry>
+    </collision>
+  </link>
+  <joint
+    name="${prefix}joint_1"
+    type="continuous">
+    <origin
+      xyz="0 0 0.1"
+      rpy="0 0 0" />
+    <parent
+      link="${prefix}base_link" />
+    <child
+      link="${prefix}link_1" />
+    <axis
+      xyz="0 0 1" />
+  </joint>
+  <link
+    name="${prefix}end_effector">
+    <inertial>
+      <origin
+        xyz="-0.0202 -0.0062674 0"
+        rpy="0 0 0" />
+      <mass
+        value="0.17604" />
+      <inertia
+        ixx="6.4514E-05"
+        ixy="-2.3173E-05"
+        ixz="-2.9024E-21"
+        iyy="0.00013201"
+        iyz="-5.9931E-22"
+        izz="0.0001392" />
+    </inertial>
+    <visual>
+      <origin
+        xyz="0 0 0"
+        rpy="0 0 0" />
+      <geometry>
+        <mesh
+          filename="package://onelink_robot/meshes/end_effector.STL" />
+      </geometry>
+      <material
+        name="">
+        <color
+          rgba="0.69412 0.098039 0.098039 1" />
+      </material>
+    </visual>
+    <collision>
+      <origin
+        xyz="0 0 0"
+        rpy="0 0 0" />
+      <geometry>
+        <mesh
+          filename="package://onelink_robot/meshes/end_effector.STL" />
+      </geometry>
+    </collision>
+  </link>
+  <joint
+    name="${prefix}joint_2"
+    type="fixed">
+    <origin
+      xyz="0.44881 0.13925 0.095"
+      rpy="0 0 0" />
+    <parent
+      link="${prefix}link_1" />
+    <child
+      link="${prefix}end_effector" />
+    <axis
+      xyz="0.95508 0.29634 0" />
+  </joint>
   </xacro:macro>
 </robot>
